Commit message: update robot pkgs

File: rsrobot_description/urdf/barista_kobuki.xacro (robot description, xacro)
@@ -33,4 +33,33 @@
       </inertial>
     </link>
+    <link name="middle_base_link">
+      <inertial>
+        <origin xyz="0.0 0.0 0.0" rpy="0.0 0.0 0.0"/>
+        <mass value="0.0"/>
+        <inertia ixx="0.0" ixy="0.0" ixz="0.0" iyy="0.0" iyz="0.0" izz="0.0"/>
+      </inertial>
+      <visual name="">
+        <origin xyz="0.0 0.0 0.0" rpy="0.0 0.0 0.0"/>
+        <geometry>
+          <cylinder radius="0.17" length="0.03"/>
+        </geometry>
+        <material name="">
+          <color rgba="1.0 0.0 0.0 1.0"/>
+          <texture filename=""/>
+        </material>
+      </visual>
+      <collision>
+        <origin xyz="0.0 0.0 0.0" rpy="0.0 0.0 0.0"/>
+        <geometry>
+           <mesh filename="package://rsrobot_description/meshes/barista/TOP_colour.dae"/>
+        </geometry>
+      </collision>
+    </link>
+    <joint name="middle_base_joint" type="fixed">
+      <parent link="base_link"/>
+      <child link="middle_base_link"/>
+      <origin xyz="0.00 0.0 0.2" rpy="0 0 0"/>
+      <axis xyz="0 0 0"/>
+    </joint>
     <link name="top_base_link">
       <inertial>
@@ -59,5 +88,5 @@
       <parent link="base_link"/>
       <child link="top_base_link"/>
-      <origin xyz="0.00 0.0 0.3" rpy="0 0 0"/>
+      <origin xyz="0.00 0.0 0.33" rpy="0 0 0"/>
       <axis xyz="0 0 0"/>
     </joint>
@@ -318,3 +347,93 @@
       <link name="camera_link_optical">
     </link>
+  <link name="ultrasonic1_link">
+    <inertial>
+      <origin xyz="0.0 0.0 0.0" rpy="0.0 0.0 0.0"/>
+      <mass value="0.0"/>
+      <inertia ixx="0.0" ixy="0.0" ixz="0.0" iyy="0.0" iyz="0.0" izz="0.0"/>
+    </inertial>
+    <visual name="">
+      <origin xyz="0.0 0.0 0.0" rpy="0.0 0.0 0.0"/>
+      <geometry>
+        <box size="0.01 0.05 0.03"/>
+      </geometry>
+      <material name="">
+        <color rgba="1.0 0.0 0.0 1.0"/>
+        <texture filename=""/>
+      </material>
+    </visual>
+    <collision>
+      <origin xyz="0.0 0.0 0.0" rpy="0.0 0.0 0.0"/>
+      <geometry>
+        <box size="0.01 0.05 0.03"/>
+      </geometry>
+    </collision>
+  </link>
+<joint name="ultrasonic1_joint" type="fixed">
+  <origin xyz="0.18 0.0 0.0" rpy="0.0 0.0 0.0"/>
+  <parent link="base_link"/>
+  <child link="ultrasonic1_link"/>
+  <axis xyz="0.0 0.0 0.0"/>
+  <limit lower="0.0" upper="0.0" effort="0.0" velocity="0.0"/>
+</joint>
+  <link name="ultrasonic2_link">
+    <inertial>
+      <origin xyz="0.0 0.0 0.0" rpy="0.0 0.0 0.0"/>
+      <mass value="0.0"/>
+      <inertia ixx="0.0" ixy="0.0" ixz="0.0" iyy="0.0" iyz="0.0" izz="0.0"/>
+    </inertial>
+    <visual name="">
+      <origin xyz="0.0 0.0 0.0" rpy="0.0 0.0 0.0"/>
+      <geometry>
+        <box size="0.01 0.05 0.03"/>
+      </geometry>
+      <material name="">
+        <color rgba="1.0 0.0 0.0 1.0"/>
+        <texture filename=""/>
+      </material>
+    </visual>
+    <collision>
+      <origin xyz="0.0 0.0 0.0" rpy="0.0 0.0 0.0"/>
+      <geometry>
+        <box size="0.01 0.05 0.03"/>
+      </geometry>
+    </collision>
+  </link>
+<joint name="ultrasonic2_joint" type="fixed">
+  <origin xyz="0.0 0.18 0.0" rpy="0.0 0.0 1.57"/>
+  <parent link="base_link"/>
+  <child link="ultrasonic2_link"/>
+  <axis xyz="0.0 0.0 0.0"/>
+  <limit lower="0.0" upper="0.0" effort="0.0" velocity="0.0"/>
+</joint>
+  <link name="ultrasonic3_link">
+    <inertial>
+      <origin xyz="0.0 0.0 0.0" rpy="0.0 0.0 0.0"/>
+      <mass value="0.0"/>
+      <inertia ixx="0.0" ixy="0.0" ixz="0.0" iyy="0.0" iyz="0.0" izz="0.0"/>
+    </inertial>
+    <visual name="">
+      <origin xyz="0.0 0.0 0.0" rpy="0.0 0.0 0.0"/>
+      <geometry>
+        <box size="0.01 0.05 0.03"/>
+      </geometry>
+      <material name="">
+        <color rgba="1.0 0.0 0.0 1.0"/>
+        <texture filename=""/>
+      </material>
+    </visual>
+    <collision>
+      <origin xyz="0.0 0.0 0.0" rpy="0.0 0.0 0.0"/>
+      <geometry>
+        <box size="0.01 0.05 0.03"/>
+      </geometry>
+    </collision>
+  </link>
+<joint name="ultrasonic3_joint" type="fixed">
+  <origin xyz="0.0 -0.18 0.0" rpy="0.0 0.0 -1.57"/>
+  <parent link="base_link"/>
+  <child link="ultrasonic3_link"/>
+  <axis xyz="0.0 0.0 0.0"/>
+  <limit lower="0.0" upper="0.0" effort="0.0" velocity="0.0"/>
+</joint>
 </robot>

Commit message: update geometry

File: rsrobot_description/urdf/barista_kobuki.xacro (robot description, xacro)
@@ -52,5 +52,5 @@
         <origin xyz="0.0 0.0 0.0" rpy="0.0 0.0 0.0"/>
         <geometry>
-           <mesh filename="package://rsrobot_description/meshes/barista/TOP_colour.dae"/>
+           <cylinder radius="0.17" length="0.03"/>
         </geometry>
       </collision>
