Commit message: fix lidar position

File: rsrobot_description/urdf/rs_real_rplidar.xacro (robot description, xacro)
@@ -178,6 +178,6 @@
   </joint>
     <joint name="laser_data_joint" type="fixed">
-      <origin xyz="0 0 0" rpy="0 -1.5707 -1.5707"/>
-      <parent link="lidar_link"/>
+      <origin xyz="0.06 0 0.19" rpy="0 0 -1.5708"/>
+      <parent link="base_link"/>
       <child link="laser_data_link"/>
     </joint>
