Commit message: fix urdf

File: rsrobot_description/urdf/rs_real.xacro (robot description, xacro)
@@ -343,10 +343,10 @@
         <origin xyz="0.11 0.0 0.23" rpy="0.0 0.0 0.0"/>
         <parent link="base_link"/>
-        <child link="kinect_link"/>
+        <child link="camera_link"/>
         <axis xyz="0.0 0 1.0"/>
       </joint>
       <joint name="camera_optical_joint" type="fixed">
         <origin xyz="0 0 0" rpy="-1.5707 0 -1.5707"/>
-        <parent link="kinect_link"/>
+        <parent link="camera_link"/>
         <child link="camera_link_optical"/>
       </joint>

Commit message: updater camera pose

File: rsrobot_description/urdf/rs_real.xacro (robot description, xacro)
@@ -341,5 +341,5 @@
     </link>
       <joint name="kinect_joint" type="fixed">
-        <origin xyz="0.11 0.0 0.23" rpy="0.0 0.0 0.0"/>
+        <origin xyz="0.05 0.0 0.22" rpy="0.0 0.0 0.0"/>
         <parent link="base_link"/>
         <child link="camera_link"/>

Commit message: update urdf and navigation

File: rsrobot_description/urdf/rs_real.xacro (robot description, xacro)
@@ -341,5 +341,5 @@
     </link>
       <joint name="kinect_joint" type="fixed">
-        <origin xyz="0.05 0.0 0.22" rpy="0.0 0.0 0.0"/>
+        <origin xyz="0.11 0.0 0.20" rpy="0.0 0.0 0.0"/>
         <parent link="base_link"/>
         <child link="camera_link"/>
@@ -353,4 +353,33 @@
       <link name="camera_link_optical">
     </link>
+  <link name="imu_link">
+    <inertial>
+      <origin xyz="0.0 0.0 0.0" rpy="0.0 0.0 0.0"/>
+      <mass value="0.0"/>
+      <inertia ixx="0.0" ixy="0.0" ixz="0.0" iyy="0.0" iyz="0.0" izz="0.0"/>
+    </inertial>
+    <visual name="">
+      <origin xyz="0.0 0.0 0.0" rpy="0.0 0.0 0.0"/>
+      <geometry>
+        <box size="0.03 0.03 0.01"/>
+      </geometry>
+      <material name="">
+        <color rgba="1.0 0.0 0.0 1.0"/>
+        <texture filename=""/>
+      </material>
+    </visual>
+    <collision>
+      <origin xyz="0.0 0.0 0.0" rpy="0.0 0.0 0.0"/>
+      <geometry>
+        <box size="0.03 0.03 0.01"/>
+      </geometry>
+    </collision>
+  </link>
+  <joint name="imu_joint" type="fixed">
+    <origin xyz="0.09 0.0 0.084" rpy="1.5707 0 0"/>
+    <parent link="base_link"/>
+    <child link="imu_link"/>
+    <axis xyz="0.0 0.0 0.0"/>
+  </joint>
   <!-- <link name="ultrasonic1_link">
     <inertial>

Commit message: update urdf

File: rsrobot_description/urdf/rs_real.xacro (robot description, xacro)
@@ -382,93 +382,3 @@
     <axis xyz="0.0 0.0 0.0"/>
   </joint>
-  <!-- <link name="ultrasonic1_link">
-    <inertial>
-      <origin xyz="0.0 0.0 0.0" rpy="0.0 0.0 0.0"/>
-      <mass value="0.0"/>
-      <inertia ixx="0.0" ixy="0.0" ixz="0.0" iyy="0.0" iyz="0.0" izz="0.0"/>
-    </inertial>
-    <visual name="">
-      <origin xyz="0.0 0.0 0.0" rpy="0.0 0.0 0.0"/>
-      <geometry>
-        <box size="0.01 0.05 0.03"/>
-      </geometry>
-      <material name="">
-        <color rgba="1.0 0.0 0.0 1.0"/>
-        <texture filename=""/>
-      </material>
-    </visual>
-    <collision>
-      <origin xyz="0.0 0.0 0.0" rpy="0.0 0.0 0.0"/>
-      <geometry>
-        <box size="0.01 0.05 0.03"/>
-      </geometry>
-    </collision>
-  </link>
-<joint name="ultrasonic1_joint" type="fixed">
-  <origin xyz="0.18 0.0 0.0" rpy="0.0 0.0 0.0"/>
-  <parent link="base_link"/>
-  <child link="ultrasonic1_link"/>
-  <axis xyz="0.0 0.0 0.0"/>
-  <limit lower="0.0" upper="0.0" effort="0.0" velocity="0.0"/>
-</joint>
-  <link name="ultrasonic2_link">
-    <inertial>
-      <origin xyz="0.0 0.0 0.0" rpy="0.0 0.0 0.0"/>
-      <mass value="0.0"/>
-      <inertia ixx="0.0" ixy="0.0" ixz="0.0" iyy="0.0" iyz="0.0" izz="0.0"/>
-    </inertial>
-    <visual name="">
-      <origin xyz="0.0 0.0 0.0" rpy="0.0 0.0 0.0"/>
-      <geometry>
-        <box size="0.01 0.05 0.03"/>
-      </geometry>
-      <material name="">
-        <color rgba="1.0 0.0 0.0 1.0"/>
-        <texture filename=""/>
-      </material>
-    </visual>
-    <collision>
-      <origin xyz="0.0 0.0 0.0" rpy="0.0 0.0 0.0"/>
-      <geometry>
-        <box size="0.01 0.05 0.03"/>
-      </geometry>
-    </collision>
-  </link>
-<joint name="ultrasonic2_joint" type="fixed">
-  <origin xyz="0.0 0.18 0.0" rpy="0.0 0.0 1.57"/>
-  <parent link="base_link"/>
-  <child link="ultrasonic2_link"/>
-  <axis xyz="0.0 0.0 0.0"/>
-  <limit lower="0.0" upper="0.0" effort="0.0" velocity="0.0"/>
-</joint>
-  <link name="ultrasonic3_link">
-    <inertial>
-      <origin xyz="0.0 0.0 0.0" rpy="0.0 0.0 0.0"/>
-      <mass value="0.0"/>
-      <inertia ixx="0.0" ixy="0.0" ixz="0.0" iyy="0.0" iyz="0.0" izz="0.0"/>
-    </inertial>
-    <visual name="">
-      <origin xyz="0.0 0.0 0.0" rpy="0.0 0.0 0.0"/>
-      <geometry>
-        <box size="0.01 0.05 0.03"/>
-      </geometry>
-      <material name="">
-        <color rgba="1.0 0.0 0.0 1.0"/>
-        <texture filename=""/>
-      </material>
-    </visual>
-    <collision>
-      <origin xyz="0.0 0.0 0.0" rpy="0.0 0.0 0.0"/>
-      <geometry>
-        <box size="0.01 0.05 0.03"/>
-      </geometry>
-    </collision>
-  </link>
-<joint name="ultrasonic3_joint" type="fixed">
-  <origin xyz="0.0 -0.18 0.0" rpy="0.0 0.0 -1.57"/>
-  <parent link="base_link"/>
-  <child link="ultrasonic3_link"/>
-  <axis xyz="0.0 0.0 0.0"/>
-  <limit lower="0.0" upper="0.0" effort="0.0" velocity="0.0"/>
-</joint> -->
 </robot>
